Commit message: simpler meshes
properly use simplified meshes to improve runtime

File: python/spot/assets/spot_simple.urdf (robot description, URDF)
Before this commit: robot spot, 15 links, 14 joints
Links:
- link body: geometry visual mesh filename=./meshes/base_simple/visual/body.obj
- link fl_hip: geometry visual mesh filename=./meshes/base_simple/visual/fl_hip.obj
- link fl_lleg: geometry visual mesh filename=./meshes/base_simple/visual/lleg.obj
- link fl_uleg: geometry visual mesh filename=./meshes/base_simple/visual/fl_uleg.obj
- link fr_hip: geometry visual mesh filename=./meshes/base_simple/visual/fr_hip.obj
- link fr_lleg: geometry visual mesh filename=./meshes/base_simple/visual/lleg.obj
- link fr_uleg: geometry visual mesh filename=./meshes/base_simple/visual/fr_uleg.obj
- link hl_hip: geometry visual mesh filename=./meshes/base_simple/visual/hl_hip.obj
- link hl_lleg: geometry visual mesh filename=./meshes/base_simple/visual/lleg.obj
- link hl_uleg: geometry visual mesh filename=./meshes/base_simple/visual/hl_uleg.obj
- link hr_hip: geometry visual mesh filename=./meshes/base_simple/visual/hr_hip.obj
- link hr_lleg: geometry visual mesh filename=./meshes/base_simple/visual/lleg.obj
- link hr_uleg: geometry visual mesh filename=./meshes/base_simple/visual/hr_uleg.obj
