Commit message: cleaning
cleanup timers and slightly decrease step callback timer

File: server/src/spot_sim/resource/spot_simple.urdf (robot description, URDF)
Before this commit: robot spot, 15 links, 14 joints
Links:
- link fl_hip: geometry visual mesh filename=./meshes/base_simple/visual/hip.obj
- link fl_uleg: geometry visual mesh filename=./meshes/base_simple/visual/uleg.obj
- link fr_hip: geometry visual mesh filename=./meshes/base_simple/visual/hip.obj
- link fr_uleg: geometry visual mesh filename=./meshes/base_simple/visual/uleg.obj
- link hl_hip: geometry visual mesh filename=./meshes/base_simple/visual/hip.obj
- link hl_uleg: geometry visual mesh filename=./meshes/base_simple/visual/uleg.obj
- link hr_hip: geometry visual mesh filename=./meshes/base_simple/visual/hip.obj
- link hr_uleg: geometry visual mesh filename=./meshes/base_simple/visual/uleg.obj
